File: Schematics/KiCad_EEG_Ver1/EEG_V1/EEG_V1.kicad_sch (KiCad schematic)
At the start: 73 parts, among them U1 INA819IDGK, U2 OPA172IDR, U3 OPA172IDR, U4 OPA172IDR, U5 OPA172IDR, U6 OPA172IDR, U7 OPA172IDR, U8 OPA172IDR, U9 OPA172IDR

Commit message: Added notch filter 50Hz
Parts:
- added C30, C31, C33, C34, C35, C36, C37, C39, C40, C41, C42, C43: 0.1u, symbol Device:C
- added C32, C38: 0.2u, symbol Device:C
- added R30, R31, R35, R37: 32k, symbol Device:R
- added R32, R36: 16k, symbol Device:R
- added R33, R39, R40: 10k, symbol Device:R
- added R34, R38: 250, symbol Device:R
- added U10, U11, U12, U13: OPA172IDR, D0008A_N, symbol EEG part lib:OPA172IDR
Connections:
- net GND: now also C33.1, C34.2, C35.1, C36.2, C40.2, C41.1, C42.1, C43.2, R33.2, R39.2, R40.2
- net V++: now also C33.2, C35.2, C41.2, C42.2, U10.7 (V+), U11.7 (V+), U12.7 (V+), U13.7 (V+)
- net V--: now also C34.1, C36.1, C40.1, C43.1, U10.4 (V-), U11.4 (V-), U12.4 (V-), U13.4 (V-)
- new net: C38.1, R36.1, U13.2 (IN-), U13.6 (OUT)
- new net: C37.2, C39.1, R36.2
- new net: R38.2, R39.1, U13.3 (IN+)
- new net: C39.2, R37.2, U12.3 (IN+)
- new net: C38.2, R35.2, R37.1
- new net: C37.1, R34.1, R35.1, U10.2 (IN-), U10.6 (OUT)
- new net: C32.1, R32.1, U11.2 (IN-), U11.6 (OUT)
- new net: R33.1, R34.2, U11.3 (IN+)
- new net: C30.2, C31.1, R32.2
- new net: R38.1, R40.1, U12.2 (IN-), U12.6 (OUT)
- new net: C32.2, R30.2, R31.1
- new net: R31.2, U10.3 (IN+)
- new net Notch_in: C30.1, R30.1
Other:
- moved on the sheet: C10, C3, C4, C5, C6, C7, C8, C9, R2, R3, R4, R5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

Commit message: Schematic update
Parts:
- added C44, C45: 0.1u, symbol Device:C
- added U14: AD8646ARZ-REEL7, R_8_ADI, symbol 2024-03-20_00-36-06:AD8646ARZ-REEL7
Connections:
- net GND: now also C44.1, C45.2
- net V++: now also C44.2, U14.8 (V+)
- net V--: now also C45.1, U14.4 (V-)
- net at C31.2: now also R31.2, U10.3 (IN+)
Other:
- added sheet Notch Filter Designs (untitled.kicad_sch)
- moved on the sheet: C30, C31, C32, C33, C34, C35, C36, C37, C38, C39, C40, C41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
