File: Schematics/KiCad_EEG_Ver1/EEG_V1/EEG_V1.kicad_sch (KiCad schematic)
At the start: 73 parts, among them U1 INA819IDGK, U2 OPA172IDR, U3 OPA172IDR, U4 OPA172IDR, U5 OPA172IDR, U6 OPA172IDR, U7 OPA172IDR, U8 OPA172IDR, U9 OPA172IDR

Commit message: Schematic update
Other:
- note added: ".tran 10m"
Changed lines of the file:
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@@
     (effects (font (size 1.27 1.27)) (justify right bottom))
+  )
+  (text ".tran 10m" (at 35.56 121.92 0)
+    (effects (font (size 1.27 1.27)) (justify left bottom))
   )
   (label "Vout1" (at 156.21 39.37 180) (fields_autoplaced)
